File: KiCad Files/ESC/ESC.kicad_pcb (KiCad board)
At the start: 2 copper layers, 97 parts, among them J1 Conn_01x03, J10 Conn_01x03, J11 Conn_01x04, J2 Conn_01x06_Female, J3 Conn_01x01, J4 Conn_01x01, J5 Conn_01x01, J6 Conn_01x03, J7 Conn_01x02, J8 Conn_01x04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

Commit message: Finished PCB v1 and Started v2
Parts:
- moved J6 198.3 mm to (82.5, 138.8), turned to 270 degrees
- moved R8 165.5 mm to (75.9, 54.6), turned to 90 degrees
- moved R22 163.5 mm to (72.1, 64.0), turned to 90 degrees
- moved C4 158.9 mm to (82.7, 52.8), turned to 0 degrees
- moved J7 155.9 mm to (68.5, 87.8), turned to 0 degrees
- moved R13 151.1 mm to (68.5, 106.4), turned to 90 degrees
- moved J11 146.3 mm to (176.3, 149.2), turned to 180 degrees
- moved R12 145.3 mm to (73.7, 98.8), turned to 270 degrees
- moved C9 145.1 mm to (95.1, 52.6), turned to 180 degrees
- moved R20 143.5 mm to (74.0, 105.0), turned to 180 degrees
- moved U3 142.5 mm to (87.3, 67.2), turned to 180 degrees
- moved R15 140.4 mm to (93.9, 59.6), turned to 0 degrees
- moved R17 139.0 mm to (76.5, 115.5), turned to 90 degrees
- moved R24 138.6 mm to (80.3, 91.3), turned to 180 degrees
- moved R23 136.0 mm to (94.3, 64.6), turned to 180 degrees
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Routing:
- net /PhaseCTrig: track 9.39 -> 40.6 mm, vias 0 -> 2
- net LogicVCC: track 273.7 -> 300.8 mm
- net /PhaseBTrig: track 16.4 -> 42.5 mm, vias 0 -> 1
- net LogicGND: track 293.6 -> 317.7 mm
- net /PhaseATrig: track 13.9 -> 37.1 mm, vias 0 -> 2
- net /HCEN: track 0.00 -> 19.0 mm
- net /HCTx: track 0.00 -> 18.7 mm
- net /HCState: track 0.00 -> 18.7 mm
- net /HCRx: track 0.00 -> 18.7 mm
- net Net-(R13-Pad1): track 101.8 -> 108.3 mm
Other:
- board outline added: 153.2 x 121.6 mm
- board text added: "1/5/18"
- board text added: "E(4)SC PCB v1"
- board text added: "L & M E(4)SC"
- board text added: "PCB for v1 of ESC made for E4"

Commit message: Added PCB v2 and reorganized code
Routing:
- added copper zone on B.Cu, net LogicGND
- added copper zone on F.Cu, net LogicGND
Changed lines of the file:
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@@
     (links 198)
     (no_connects 18)
-    (area 59.724999 34.924999 213.075001 156.675001)
+    (area 59.724999 34.924999 215.428571 194.55)
     (thickness 1.6)
     (drawings 8)
@@
     (0 F.Cu signal)
     (31 B.Cu signal)
-    (32 B.Adhes user)
-    (33 F.Adhes user)
-    (34 B.Paste user)
-    (35 F.Paste user)
+    (32 B.Adhes user hide)
+    (33 F.Adhes user hide)
+    (34 B.Paste user hide)
+    (35 F.Paste user hide)
     (36 B.SilkS user)
     (37 F.SilkS user)
     (38 B.Mask user)
     (39 F.Mask user)
-    (40 Dwgs.User user)
+    (40 Dwgs.User user hide)
     (41 Cmts.User user)
     (42 Eco1.User user)
@@
     (visible_elements FFFFF77F)
     (pcbplotparams
-      (layerselection 0x00030_80000001)
+      (layerselection 0x000c0_80000001)
       (usegerberextensions false)
       (excludeedgelayer true)
@@
       (plotreference true)
       (plotvalue true)
-      (plotinvisibletext false)
-      (padsonsilk false)
+      (plotinvisibletext true)
+      (padsonsilk true)
       (subtractmaskfromsilk false)
-      (outputformat 1)
+      (outputformat 4)
       (mirror false)
-      (drillshape 1)
+      (drillshape 0)
       (scaleselection 1)
       (outputdirectory ""))
@@
   (segment (start 170.041724 82.527208) (end 170.001724 82.487208) (width 1.5) (layer B.Cu) (net 70))
   (segment (start 177.341724 108.937207) (end 177.341724 114.027208) (width 1.5) (layer F.Cu) (net 70))
+  (zone (net 2) (net_name LogicGND) (layer F.Cu) (hatch edge 0.508)
+    (connect_pads (clearance 0.508))
+    (min_thickness 0.254)
+    (fill yes (arc_segments 16) (thermal_gap 0.508) (thermal_bridge_width 0.508))
+    (polygon
+      (pts
+        (xy 213 156.6) (xy 59.8 156.6) (xy 59.8 35) (xy 213 35)
+      )
+    )
+  )
+  (zone (net 2) (net_name LogicGND) (layer B.Cu) (hatch edge 0.508)
+    (connect_pads (clearance 0.508))
+    (min_thickness 0.254)
+    (fill yes (arc_segments 16) (thermal_gap 0.508) (thermal_bridge_width 0.508))
+    (polygon
+      (pts
+        (xy 213 156.6) (xy 59.8 156.6) (xy 59.8 35) (xy 213 35)
+      )
+    )
+  )
 )
