File: KiCad Files/ESC/ESC.sch (KiCad schematic (older format))
At the start: 89 parts, among them J1 Conn_01x22_Male, J2 Conn_01x06_Female, J3 Screw_Terminal_01x03, Q1 IRF3205, Q2 IRF3205, Q3 IRF3205, Q4 IRF3205, Q5 IRF3205, Q6 IRF3205, U1 LM339, U2 L7809, U3 MCP601-xP, U4 IR2110, U5 IR2110, U6 IR2110

Commit message: Updated v1 of PCB
Parts:
- removed C21, C22, C23: 1u, symbol CP1_Small
- removed J1: Conn_01x22_Male, symbol Conn_01x22_Male
- removed J3: Screw_Terminal_01x03, symbol Screw_Terminal_01x03
- added C21, C22, C23: 2.2u, Capacitors_THT:C_Rect_L7.2mm_W11.0mm_P5.00mm_FKS2_FKP2_MKS2_MKP2, symbol C_Small
- added J1, J10, J6, J9: Conn_01x03, Socket_Strips:Socket_Strip_Straight_1x03_Pitch2.54mm, symbol Conn_01x03
- added J11, J8: Conn_01x04, Socket_Strips:Socket_Strip_Straight_1x04_Pitch2.54mm, symbol Conn_01x04
- added J3, J4, J5: Conn_01x01, Mounting_Holes:MountingHole_4.3mm_M4_Pad, symbol Conn_01x01
- added J7: Conn_01x02, Socket_Strips:Socket_Strip_Straight_1x02_Pitch2.54mm, symbol Conn_01x02
- 10k1: footprint (none) -> Potentiometers:Potentiometer_WirePads_Small
- BT1: footprint (none) -> Wire_Connections_Bridges:WireConnection_2.50mmDrill_LargePad
- C1: footprint (none) -> Capacitors_THT:CP_Radial_D4.0mm_P2.00mm
- C10, C9: footprint (none) -> Capacitors_THT:C_Disc_D8.0mm_W5.0mm_P5.00mm
- C11: value 6.3n -> 6.8n; footprint (none) -> Capacitors_THT:C_Disc_D8.0mm_W2.5mm_P5.00mm
- C12, C13, C14: footprint (none) -> Capacitors_THT:C_Disc_D7.5mm_W5.0mm_P5.00mm
- C15, C16, C17, C4, C5, C6, C7, C8: footprint (none) -> Capacitors_THT:C_Disc_D3.0mm_W1.6mm_P2.50mm
- C18, C19, C20: value 0.68u -> 1u; footprint (none) -> Capacitors_THT:C_Disc_D4.3mm_W1.9mm_P5.00mm
- C2: footprint (none) -> Capacitors_THT:C_Rect_L7.0mm_W2.5mm_P5.00mm
- C3: footprint (none) -> Capacitors_THT:CP_Radial_D12.5mm_P7.50mm
- D2, D3, D4: footprint (none) -> Diodes_THT:D_DO-35_SOD27_P7.62mm_Horizontal
- F1: footprint (none) -> Fuse_Holders_and_Fuses:Fuseholder_ATO_Blade_littlefuse_Pudenz_2_Pin
- F2: footprint (none) -> Fuse_Holders_and_Fuses:Fuseholder5x20_horiz_open_inline_Type-I
- J2: footprint (none) -> Socket_Strips:Socket_Strip_Angled_1x06_Pitch2.54mm
- JP1: footprint (none) -> Capacitors_Tantalum_SMD:CP_Tantalum_Case-A_EIA-3216-18_Hand
- Q1, Q2, Q3, Q4, Q5, Q6: footprint TO_SOT_Packages_THT:TO-220_Vertical -> Power_Integrations:TO-220
- R1, R10, R11, R12, R13, R14, R15, R16, R17, R18, R19, R2, R20, R22, R23, R24, R25, R26, R27, R28, R29, R3, R30, R31, R32, R33, R34, R35, R36, R37, R38, R39, R4, R40, R41, R42, R5, R6, R7, R8, R9: footprint (none) -> Resistors_SMD:R_1206_HandSoldering
- R21: footprint (none) -> Resistors_THT:R_Axial_Power_L25.0mm_W9.0mm_P30.48mm
- U1: footprint (none) -> Housings_DIP:DIP-14_W7.62mm_Socket
- U2: footprint (none) -> TO_SOT_Packages_THT:TO-220-3_Vertical
- U3: footprint (none) -> Housings_DIP:DIP-8_W7.62mm_Socket
Connections:
- net BatVoltMeas: now also J8.2 (Pin_2)
- net HCEN: now also J11.1 (Pin_1)
- net HCRx: now also J11.3 (Pin_3)
- net HCState: now also J11.4 (Pin_4)
- net HCTx: now also J11.2 (Pin_2)
- net Logic9V: now also J8.4 (Pin_4)
- net LogicGND: now also J8.3 (Pin_3)
- net LogicVCC: now also J8.1 (Pin_1)
- net MeanCur: now also J7.1 (Pin_1)
- net OverCurInt: now also J7.2 (Pin_2)
- net PhaseAHIN: now also J9.3 (Pin_3)
- net PhaseALIN: now also J9.1 (Pin_1)
- net PhaseASD: now also J9.2 (Pin_2)
- net PhaseATrig: now also J6.3 (Pin_3)
- net PhaseBHIN: now also J1.3 (Pin_3)
- net PhaseBLIN: now also J1.1 (Pin_1)
- net PhaseBSD: now also J1.2 (Pin_2)
- net PhaseBTrig: now also J6.2 (Pin_2)
- net PhaseCHIN: now also J10.3 (Pin_3)
- net PhaseCLIN: now also J10.1 (Pin_1)
- net PhaseCSD: now also J10.2 (Pin_2)
- net PhaseCTrig: now also J6.1 (Pin_1)
- net PowerGND: now also C21.2, C22.2, C23.2
- net PowerVCC: now also C21.1, C22.1, C23.1; no longer C18.2, C19.2, C20.2, Q1.3 (S), Q2.2 (D), Q3.3 (S), Q4.2 (D), Q5.3 (S), Q6.2 (D), R11.2, R16.2, R19.2, R25.1, R27.1, R28.1, R37.2, R38.2, R39.2, U4.5 (VS), U5.5 (VS), U6.5 (VS)
- new net PhaseA: C18.2, J3.1 (Pin_1), Q1.3 (S), Q2.2 (D), R19.2, R28.1, R37.2, U4.5 (VS)
- new net PhaseB: C19.2, J4.1 (Pin_1), Q3.3 (S), Q4.2 (D), R16.2, R27.1, R38.2, U5.5 (VS)
- new net PhaseC: C20.2, J5.1 (Pin_1), Q5.3 (S), Q6.2 (D), R11.2, R25.1, R39.2, U6.5 (VS)
Other:
- note added: "Basic BLDC controller with current measuring capabilities and bluetooth communication, \nfor use with MAX32 Kit.\nProject made for Eletrónica 4 @ UA"
- note removed: "MCP601 e MCP6021\ntem o mesmo pinout,\nexcepto o pin 5, que \nno 6021 corresponde a\nVREF e no 601 está\nNC"

Commit message: Finished PCB v1 and Started v2
Changed lines of the file:
@@
 	10650 2350 6100 2350
 Wire Notes Line
-	850  1750 850  4300
-Wire Notes Line
-	850  4300 2300 4300
+	500  4300 2300 4300
 Wire Notes Line
 	850  550  4150 550
@@
 	-1   0    0    1
 $EndComp
+Wire Notes Line
+	500  4300 500  1750
+Wire Notes Line
+	500  1750 900  1750
 $EndSCHEMATC

Commit message: Added PCB v2 and reorganized code
Parts:
- C10, C9: footprint Capacitors_THT:C_Disc_D8.0mm_W5.0mm_P5.00mm -> Capacitors_SMD:C_1206_HandSoldering
- C11: footprint Capacitors_THT:C_Disc_D8.0mm_W2.5mm_P5.00mm -> Capacitors_SMD:C_1206_HandSoldering
- C12, C13, C14: footprint Capacitors_THT:C_Disc_D7.5mm_W5.0mm_P5.00mm -> Capacitors_SMD:C_1206_HandSoldering
- C15, C16, C17, C4, C5, C6, C7, C8: footprint Capacitors_THT:C_Disc_D3.0mm_W1.6mm_P2.50mm -> Capacitors_SMD:C_1206_HandSoldering
- C18, C19, C20: footprint Capacitors_THT:C_Disc_D4.3mm_W1.9mm_P5.00mm -> Capacitors_SMD:C_1206_HandSoldering
- C2: value 82n -> 100n; footprint Capacitors_THT:C_Rect_L7.0mm_W2.5mm_P5.00mm -> Capacitors_SMD:C_1206_HandSoldering
- C21, C22, C23: value 2.2u -> 1u; footprint Capacitors_THT:C_Rect_L7.2mm_W11.0mm_P5.00mm_FKS2_FKP2_MKS2_MKP2 -> Capacitors_THT:C_Disc_D4.3mm_W1.9mm_P5.00mm
Changed lines of the file:
@@
 F 0 "C18" H 8160 1470 50  0000 L CNN
 F 1 "1u" H 8160 1320 50  0000 L CNN
-F 2 "Capacitors_THT:C_Disc_D4.3mm_W1.9mm_P5.00mm" H 8150 1400 50  0001 C CNN
+F 2 "Capacitors_SMD:C_1206_HandSoldering" H 8150 1400 50  0001 C CNN
 F 3 "" H 8150 1400 50  0001 C CNN
 	1    8150 1400
@@
 F 0 "C15" H 7960 1970 50  0000 L CNN
 F 1 "33n" H 7960 1820 50  0000 L CNN
-F 2 "Capacitors_THT:C_Disc_D3.0mm_W1.6mm_P2.50mm" H 7950 1900 50  0001 C CNN
+F 2 "Capacitors_SMD:C_1206_HandSoldering" H 7950 1900 50  0001 C CNN
 F 3 "" H 7950 1900 50  0001 C CNN
 	1    7950 1900
@@
 F 0 "C12" H 6910 1220 50  0000 L CNN
 F 1 "10n" H 6910 1070 50  0000 L CNN
-F 2 "Capacitors_THT:C_Disc_D7.5mm_W5.0mm_P5.00mm" H 6900 1150 50  0001 C CNN
+F 2 "Capacitors_SMD:C_1206_HandSoldering" H 6900 1150 50  0001 C CNN
 F 3 "" H 6900 1150 50  0001 C CNN
 	1    6900 1150
@@
 P 2800 1100
 F 0 "C2" H 2810 1170 50  0000 L CNN
-F 1 "82n" H 2810 1020 50  0000 L CNN
-F 2 "Capacitors_THT:C_Rect_L7.0mm_W2.5mm_P5.00mm" H 2800 1100 50  0001 C CNN
+F 1 "100n" H 2810 1020 50  0000 L CNN
+F 2 "Capacitors_SMD:C_1206_HandSoldering" H 2800 1100 50  0001 C CNN
 F 3 "" H 2800 1100 50  0001 C CNN
 	1    2800 1100
@@
 F 0 "C19" H 8160 3320 50  0000 L CNN
 F 1 "1u" H 8160 3170 50  0000 L CNN
-F 2 "Capacitors_THT:C_Disc_D4.3mm_W1.9mm_P5.00mm" H 8150 3250 50  0001 C CNN
+F 2 "Capacitors_SMD:C_1206_HandSoldering" H 8150 3250 50  0001 C CNN
 F 3 "" H 8150 3250 50  0001 C CNN
 	1    8150 3250
@@
 F 0 "C16" H 7960 3820 50  0000 L CNN
 F 1 "33n" H 7960 3670 50  0000 L CNN
-F 2 "Capacitors_THT:C_Disc_D3.0mm_W1.6mm_P2.50mm" H 7950 3750 50  0001 C CNN
+F 2 "Capacitors_SMD:C_1206_HandSoldering" H 7950 3750 50  0001 C CNN
 F 3 "" H 7950 3750 50  0001 C CNN
 	1    7950 3750
@@
 F 0 "C13" H 6910 3070 50  0000 L CNN
 F 1 "10n" H 6910 2920 50  0000 L CNN
-F 2 "Capacitors_THT:C_Disc_D7.5mm_W5.0mm_P5.00mm" H 6900 3000 50  0001 C CNN
+F 2 "Capacitors_SMD:C_1206_HandSoldering" H 6900 3000 50  0001 C CNN
 F 3 "" H 6900 3000 50  0001 C CNN
 	1    6900 3000
@@
 F 0 "C20" H 8160 5170 50  0000 L CNN
 F 1 "1u" H 8160 5020 50  0000 L CNN
-F 2 "Capacitors_THT:C_Disc_D4.3mm_W1.9mm_P5.00mm" H 8150 5100 50  0001 C CNN
+F 2 "Capacitors_SMD:C_1206_HandSoldering" H 8150 5100 50  0001 C CNN
 F 3 "" H 8150 5100 50  0001 C CNN
 	1    8150 5100
@@
 F 0 "C17" H 7960 5670 50  0000 L CNN
 F 1 "33n" H 7960 5520 50  0000 L CNN
-F 2 "Capacitors_THT:C_Disc_D3.0mm_W1.6mm_P2.50mm" H 7950 5600 50  0001 C CNN
+F 2 "Capacitors_SMD:C_1206_HandSoldering" H 7950 5600 50  0001 C CNN
 F 3 "" H 7950 5600 50  0001 C CNN
 	1    7950 5600
@@
 F 0 "C14" H 6910 4920 50  0000 L CNN
 F 1 "10n" H 6910 4770 50  0000 L CNN
-F 2 "Capacitors_THT:C_Disc_D7.5mm_W5.0mm_P5.00mm" H 6900 4850 50  0001 C CNN
+F 2 "Capacitors_SMD:C_1206_HandSoldering" H 6900 4850 50  0001 C CNN
 F 3 "" H 6900 4850 50  0001 C CNN
 	1    6900 4850
@@
 F 0 "C11" H 6310 7470 50  0000 L CNN
 F 1 "6.8n" H 6310 7320 50  0000 L CNN
-F 2 "Capacitors_THT:C_Disc_D8.0mm_W2.5mm_P5.00mm" H 6300 7400 50  0001 C CNN
+F 2 "Capacitors_SMD:C_1206_HandSoldering" H 6300 7400 50  0001 C CNN
 F 3 "" H 6300 7400 50  0001 C CNN
 	1    6300 7400
@@
 F 0 "C8" H 4210 7120 50  0000 L CNN
 F 1 "1n" H 4210 6970 50  0000 L CNN
-F 2 "Capacitors_THT:C_Disc_D3.0mm_W1.6mm_P2.50mm" H 4200 7050 50  0001 C CNN
+F 2 "Capacitors_SMD:C_1206_HandSoldering" H 4200 7050 50  0001 C CNN
 F 3 "" H 4200 7050 50  0001 C CNN
 	1    4200 7050
@@
 F 0 "C7" H 3860 7120 50  0000 L CNN
 F 1 "1n" H 3860 6970 50  0000 L CNN
-F 2 "Capacitors_THT:C_Disc_D3.0mm_W1.6mm_P2.50mm" H 3850 7050 50  0001 C CNN
+F 2 "Capacitors_SMD:C_1206_HandSoldering" H 3850 7050 50  0001 C CNN
 F 3 "" H 3850 7050 50  0001 C CNN
 	1    3850 7050
@@
 F 0 "C5" H 3510 7120 50  0000 L CNN
 F 1 "1n" H 3510 6970 50  0000 L CNN
-F 2 "Capacitors_THT:C_Disc_D3.0mm_W1.6mm_P2.50mm" H 3500 7050 50  0001 C CNN
+F 2 "Capacitors_SMD:C_1206_HandSoldering" H 3500 7050 50  0001 C CNN
 F 3 "" H 3500 7050 50  0001 C CNN
 	1    3500 7050
@@
 F 0 "C9" H 4610 1220 50  0000 R CNN
 F 1 "5.6n" H 4610 1070 50  0000 R CNN
-F 2 "Capacitors_THT:C_Disc_D8.0mm_W5.0mm_P5.00mm" H 4600 1150 50  0001 C CNN
+F 2 "Capacitors_SMD:C_1206_HandSoldering" H 4600 1150 50  0001 C CNN
 F 3 "" H 4600 1150 50  0001 C CNN
 	1    4600 1150
@@
 F 0 "C10" H 5760 1770 50  0000 L CNN
 F 1 "5.6n" H 5760 1620 50  0000 L CNN
-F 2 "Capacitors_THT:C_Disc_D8.0mm_W5.0mm_P5.00mm" H 5750 1700 50  0001 C CNN
+F 2 "Capacitors_SMD:C_1206_HandSoldering" H 5750 1700 50  0001 C CNN
 F 3 "" H 5750 1700 50  0001 C CNN
 	1    5750 1700
@@
 F 0 "C4" H 3510 2420 50  0000 L CNN
 F 1 "33n" H 3510 2270 50  0000 L CNN
-F 2 "Capacitors_THT:C_Disc_D3.0mm_W1.6mm_P2.50mm" H 3500 2350 50  0001 C CNN
+F 2 "Capacitors_SMD:C_1206_HandSoldering" H 3500 2350 50  0001 C CNN
 F 3 "" H 3500 2350 50  0001 C CNN
 	1    3500 2350
@@
 F 0 "C6" H 3710 1170 50  0000 L CNN
 F 1 "1n" H 3710 1020 50  0000 L CNN
-F 2 "Capacitors_THT:C_Disc_D3.0mm_W1.6mm_P2.50mm" H 3700 1100 50  0001 C CNN
+F 2 "Capacitors_SMD:C_1206_HandSoldering" H 3700 1100 50  0001 C CNN
 F 3 "" H 3700 1100 50  0001 C CNN
 	1    3700 1100
@@
 P 9800 1250
 F 0 "C21" H 9810 1320 50  0000 L CNN
-F 1 "2.2u" H 9810 1170 50  0000 L CNN
-F 2 "Capacitors_THT:C_Rect_L7.2mm_W11.0mm_P5.00mm_FKS2_FKP2_MKS2_MKP2" H 9800 1250 50  0001 C CNN
+F 1 "1u" H 9810 1170 50  0000 L CNN
+F 2 "Capacitors_THT:C_Disc_D4.3mm_W1.9mm_P5.00mm" H 9800 1250 50  0001 C CNN
 F 3 "" H 9800 1250 50  0001 C CNN
 	1    9800 1250
@@
 P 9800 3100
 F 0 "C22" H 9810 3170 50  0000 L CNN
-F 1 "2.2u" H 9810 3020 50  0000 L CNN
-F 2 "Capacitors_THT:C_Rect_L7.2mm_W11.0mm_P5.00mm_FKS2_FKP2_MKS2_MKP2" H 9800 3100 50  0001 C CNN
+F 1 "1u" H 9810 3020 50  0000 L CNN
+F 2 "Capacitors_THT:C_Disc_D4.3mm_W1.9mm_P5.00mm" H 9800 3100 50  0001 C CNN
 F 3 "" H 9800 3100 50  0001 C CNN
 	1    9800 3100
@@
 P 9800 4950
 F 0 "C23" H 9810 5020 50  0000 L CNN
-F 1 "2.2u" H 9810 4870 50  0000 L CNN
-F 2 "Capacitors_THT:C_Rect_L7.2mm_W11.0mm_P5.00mm_FKS2_FKP2_MKS2_MKP2" H 9800 4950 50  0001 C CNN
+F 1 "1u" H 9810 4870 50  0000 L CNN
+F 2 "Capacitors_THT:C_Disc_D4.3mm_W1.9mm_P5.00mm" H 9800 4950 50  0001 C CNN
 F 3 "" H 9800 4950 50  0001 C CNN
 	1    9800 4950
