File: KiCad Files/ESC.kicad_pcb (KiCad board)
At the start: 2 copper layers, 110.8 x 108.2 mm, 98 parts, among them J1 Conn_01x03, J10 Conn_01x03, J3 Conn_01x01, J4 Conn_01x01, J5 Conn_01x01, J6 Conn_01x03, J7 Conn_01x02, J8 Conn_01x04, J9 Conn_01x03, Q1 IRF3205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

Commit message: Added final PCB
Parts:
- added C24: 100n, Capacitors_SMD:C_1206_HandSoldering, B.Cu at (93.0, 77.2)
- added R43: 3.3k, Resistors_SMD:R_1206_HandSoldering, B.Cu at (96.8, 77.2)
- added R44: 8.2k, Resistors_SMD:R_1206_HandSoldering, B.Cu at (84.4, 74.2)
Connections:
- C2 pad 1: BatVoltMeas -> Net-(C2-Pad1)
- F2 pad 1: BatVoltMeas -> Net-(C2-Pad1)
- U2 pad 1: BatVoltMeas -> Net-(C2-Pad1)
Routing:
- net Net-(C2-Pad1): track 0.00 -> 29.5 mm
- net BatVoltMeas: track 40.4 -> 15.8 mm
- net LogicGND: track 174.7 -> 184.5 mm
Other:
- board text removed: "1/5/18"
- board text removed: "E(4)SC PCB v1"
- board text removed: "PCB v2 of ESC made for E4"
